File: resource/pcb/Micromouse/Micromouse v4.sch (EAGLE design)
At the start: 8 parts

Commit message: Updated PCB
Signed-off-by: AJ Walter <git@awalter.net>
Connections:
- new net N$1: 12V_BOOST.ENABLE, ESP1.12/A11
Changed lines of the file:
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@@
+</segment>
+</net>
+<net name="N$1" class="0">
+<segment>
+<pinref part="ESP1" gate="G$1" pin="12/A11"/>
+<wire x1="63.5" y1="50.8" x2="86.36" y2="50.8" width="0.1524" layer="91"/>
+<wire x1="86.36" y1="50.8" x2="86.36" y2="-15.24" width="0.1524" layer="91"/>
+<wire x1="86.36" y1="-15.24" x2="-50.8" y2="-15.24" width="0.1524" layer="91"/>
+<pinref part="12V_BOOST" gate="G$1" pin="ENABLE"/>
+<wire x1="-50.8" y1="-15.24" x2="-50.8" y2="73.66" width="0.1524" layer="91"/>
+<wire x1="-50.8" y1="73.66" x2="-58.42" y2="73.66" width="0.1524" layer="91"/>
 </segment>
 </net>
